File: AKS-Arduino.kicad_pcb (KiCad board)
At the start: 2 copper layers, 122.1 x 102.8 mm, 17 parts, among them J1 Jack-DC, J2 Conn_01x07_Socket, J3 Conn_01x07_Socket, J5 Conn_01x05_Socket, U1 ATmega328-P, Y1 Crystal

Commit message: Images added
Other:
- board size 122.1 x 102.8 mm -> 109.6 x 102.8 mm
- board text added: "LoRa"
- board text added: "MCP2515"
Changed lines of the file:
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@@
 		(tags "LED")
 		(property "Reference" "D5"
-			(at 1.27 -2.96 360)
+			(at 1.27 -2.96 0)
 			(layer "F.SilkS")
 			(effects
@@
 		)
 		(property "Value" "LED"
-			(at 1.27 2.96 360)
+			(at 1.27 2.96 0)
 			(layer "F.Fab")
 			(effects
@@
 		)
 		(property "Footprint" "LED_THT:LED_D3.0mm"
-			(at 0 0 360)
+			(at 0 0 0)
 			(layer "F.Fab")
 			(hide yes)
@@
 		)
 		(property "Datasheet" ""
-			(at 0 0 360)
+			(at 0 0 0)
 			(layer "F.Fab")
 			(hide yes)
@@
 		)
 		(property "Description" "Light emitting diode"
-			(at 0 0 360)
+			(at 0 0 0)
 			(layer "F.Fab")
 			(hide yes)
@@
 		)
 		(fp_text user "${REFERENCE}"
-			(at 1.11 0.23 360)
+			(at 1.11 0.23 0)
 			(layer "F.Fab")
 			(effects
@@
 		(tags "LED")
 		(property "Reference" "D6"
-			(at 1.27 -2.96 360)
+			(at 1.27 -2.96 0)
 			(layer "F.SilkS")
 			(effects
@@
 		)
 		(property "Value" "LED"
-			(at 1.27 2.96 360)
+			(at 1.27 2.96 0)
 			(layer "F.Fab")
 			(effects
@@
 		)
 		(property "Footprint" "LED_THT:LED_D3.0mm"
-			(at 0 0 360)
+			(at 0 0 0)
 			(layer "F.Fab")
 			(hide yes)
@@
 		)
 		(property "Datasheet" ""
-			(at 0 0 360)
+			(at 0 0 0)
 			(layer "F.Fab")
 			(hide yes)
@@
 		)
 		(property "Description" "Light emitting diode"
-			(at 0 0 360)
+			(at 0 0 0)
 			(layer "F.Fab")
 			(hide yes)
@@
 		)
 		(fp_text user "${REFERENCE}"
-			(at 1.27 0 360)
+			(at 1.27 0 0)
 			(layer "F.Fab")
 			(effects
@@
 		(tags "LED")
 		(property "Reference" "D4"
-			(at 1.27 -2.96 360)
+			(at 1.27 -2.96 0)
 			(layer "F.SilkS")
 			(effects
@@
 		)
 		(property "Value" "LED"
-			(at 1.27 2.96 360)
+			(at 1.27 2.96 0)
 			(layer "F.Fab")
 			(effects
@@
 		)
 		(property "Footprint" "LED_THT:LED_D3.0mm"
-			(at 0 0 360)
+			(at 0 0 0)
 			(layer "F.Fab")
 			(hide yes)
@@
 		)
 		(property "Datasheet" ""
-			(at 0 0 360)
+			(at 0 0 0)
 			(layer "F.Fab")
 			(hide yes)
@@
 		)
 		(property "Description" "Light emitting diode"
-			(at 0 0 360)
+			(at 0 0 0)
 			(layer "F.Fab")
 			(hide yes)
@@
 		)
 		(fp_text user "${REFERENCE}"
-			(at 1.27 0 360)
+			(at 1.27 0 0)
 			(layer "F.Fab")
 			(effects
@@
 	)
 	(gr_rect
-		(start 101.975 33.79)
+		(start 145.73 34.2)
+		(end 164.55 79.65)
+		(stroke
+			(width 0.2)
+			(type default)
+		)
+		(fill none)
+		(layer "F.Cu")
+	)
+	(gr_rect
+		(start 178.37 102.83)
+		(end 223.62 121.62)
+		(stroke
+			(width 0.2)
+			(type default)
+		)
+		(fill none)
+		(layer "F.Cu")
+	)
+	(gr_rect
+		(start 114.405 33.79)
 		(end 224.045 136.54)
 		(stroke
@@
 		(layer "Edge.Cuts")
 	)
+	(gr_text "MCP2515"
+		(at 198.88 112.77 0)
+		(layer "F.Cu")
+		(effects
+			(font
+				(size 1.5 1.5)
+				(thickness 0.3)
+				(bold yes)
+			)
+			(justify left bottom)
+		)
+	)
+	(gr_text "LoRa"
+		(at 152.2 38.86 0)
+		(layer "F.Cu")
+		(effects
+			(font
+				(size 1.5 1.5)
+				(thickness 0.3)
+				(bold yes)
+			)
+			(justify left bottom)
+		)
+	)
 	(segment

Commit message: Update
Parts:
- added C3: C_Polarized_US, Capacitor_THT:CP_Radial_D8.0mm_P2.50mm, F.Cu at (195.3, 82.9)
- added J4: Conn_01x02_Socket, Connector_PinSocket_2.54mm:PinSocket_1x02_P2.54mm_Vertical, F.Cu at (198.7, 39.2)
- added R3: R, Resistor_THT:R_Axial_DIN0207_L6.3mm_D2.5mm_P5.08mm_Vertical, F.Cu at (183.8, 78.1)
- moved D3 34.3 mm to (221.9, 61.8)
- moved D4 34.3 mm to (221.9, 53.8)
- moved D5 34.3 mm to (221.9, 45.8)
- moved D6 34.3 mm to (221.9, 37.8)
- moved D1 34.3 mm to (221.9, 77.8)
- moved D2 34.3 mm to (221.9, 69.8)
- moved J1 33.0 mm to (130.2, 39.9)
Connections:
- U1 pad 1: unconnected-(U1-~{RESET}/PC6-Pad1) -> RESET
Routing:
- net GND: track 271.0 -> 403.6 mm
- net RESET: track 0.00 -> 78.9 mm
- net Net-(D4-A): track 30.1 -> 80.1 mm
- net Net-(D3-A): track 26.3 -> 76.3 mm
- net Net-(D5-A): track 34.4 -> 83.5 mm
- net Net-(D6-A): track 38.0 -> 87.1 mm
- net Net-(D2-A): track 24.0 -> 72.4 mm
- net Net-(D1-A): track 21.7 -> 68.6 mm
- net +5V: track 228.8 -> 264.8 mm
- net Net-(U2-IN+): track 15.8 -> 48.5 mm
- net Net-(U2-IN-): track 14.8 -> 45.8 mm
Other:
- board text added: "AYTUNÇ TUNÇAY EREN TURHAN"

Commit message: Version 1 Last Update
Parts:
- removed D1, D2, D3, D4: LED, LED_THT:LED_D3.0mm
- added J6: Conn_01x03_Socket, Connector_PinHeader_2.54mm:PinHeader_1x03_P2.54mm_Vertical, F.Cu at (217.6, 91.2)
- added J7: Conn_01x04_Socket, Connector_PinSocket_2.54mm:PinSocket_1x04_P2.54mm_Vertical, F.Cu at (216.4, 131.3)
- added R4: R, Resistor_THT:R_Axial_DIN0207_L6.3mm_D2.5mm_P5.08mm_Vertical, F.Cu at (216.7, 80.7)
- added R5: R, Resistor_THT:R_Axial_DIN0207_L6.3mm_D2.5mm_P5.08mm_Vertical, F.Cu at (210.0, 80.8)
- moved D6 22.5 mm to (222.0, 60.3)
- moved J1 22.5 mm to (130.3, 62.4)
- moved D5 22.5 mm to (222.0, 68.3)
- moved J4 19.8 mm to (198.8, 59.1)
Connections:
- U1 pad 23: Net-(D1-A) -> Nextion TX
- U1 pad 24: Net-(D2-A) -> Nextion RX
- U1 pad 25: Net-(D3-A) -> Serial RX
- U1 pad 26: Net-(D4-A) -> Serial TX
- U1 pad 27: Net-(D5-A) -> Net-(U1-PC4)
- U1 pad 28: Net-(D6-A) -> Net-(U1-PC5)
Routing:
- net Net-(D4-A): track 80.1 -> 0.00 mm
- net Nextion RX: track 0.00 -> 77.1 mm
- net Net-(D3-A): track 76.3 -> 0.00 mm
- net Net-(D5-A): track 83.5 -> 8.40 mm
- net Nextion TX: track 0.00 -> 72.7 mm
- net Net-(D2-A): track 72.4 -> 0.00 mm
- net Net-(D1-A): track 68.6 -> 0.00 mm
- net Net-(D6-A): track 87.1 -> 19.3 mm
- net Net-(U1-PC4): track 0.00 -> 50.0 mm
- net Serial RX: track 0.00 -> 49.7 mm
- net Serial TX: track 0.00 -> 48.6 mm
- net Net-(U1-PC5): track 0.00 -> 43.0 mm
- net +5V: track 264.8 -> 298.9 mm
- net Net-(U2-IN+): track 48.5 -> 25.9 mm
- net Net-(U2-IN-): track 45.8 -> 23.3 mm
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Other:
- board size 109.6 x 102.8 mm -> 109.6 x 84 mm
- board text removed: "LoRa"
- board text removed: "MCP2515"
